File: rev5b-pcb/ecad_src/Flatbox-rev5B.kicad_pcb (KiCad board)
At the start: 2 copper layers, 210 x 120 mm, 32 parts, among them SW1 SW_Push, SW10 SW_Push, SW11 SW_Push, SW12 SW_Push, SW13 SW_Push, SW14 SW_Push, SW15 SW_Push, SW16 SW_Push, SW17 SW_Push, SW18 SW_Push, SW1_B1 SW_Push, SW2 SW_Push, SW3 SW_Push, SW3_B1 SW_Push, SW4 SW_Push, SW5 SW_Push, SW6 SW_Push, SW7 SW_Push, SW8 SW_Push, SW9 SW_Push

Commit message: 5B update
Routing:
- added copper zone on F.Cu, net GND
Other:
- board text added: "Flatbox5B"
- board text added: "github.com/nbovee/flatbox-sf6-buttons based off of: github.com/jfedor2/flatbox"
- board text removed: "Flatbox"
- board text removed: "github.com/nbovee/flatbox"
- board text removed: "rev5.B"
Changed lines of the file:
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@@
     (effects (font (size 1 1) (thickness 0.15)))
   )
-  (gr_text "rev5.B" (at 82 143) (layer "F.SilkS")
+  (gr_text "github.com/nbovee/flatbox-sf6-buttons\nbased off of: github.com/jfedor2/flatbox" (at 80.01 132.588) (layer "F.SilkS")
     (effects (font (size 2 2) (thickness 0.3)))
   )
-  (gr_text "github.com/nbovee/flatbox" (at 196 143) (layer "F.SilkS")
-    (effects (font (size 2 2) (thickness 0.3)))
-  )
-  (gr_text "Flatbox" (at 80 110) (layer "F.SilkS")
+  (gr_text "Flatbox5B" (at 78.994 124.714) (layer "F.SilkS")
     (effects (font (size 8 8) (thickness 1)))
   )
@@
   (segment (start 194.7744 123.829) (end 192.661111 123.829) (width 0.254) (layer "B.Cu") (net 27))
   (segment (start 202.493111 112.836) (end 202.493111 116.110289) (width 0.254) (layer "B.Cu") (net 27))
-  (zone (net 1) (net_name "GND") (layer "B.Cu") (hatch edge 0.508)
+  (zone (net 1) (net_name "GND") (layers "F&B.Cu") (hatch edge 0.508)
     (connect_pads (clearance 0.508))
     (min_thickness 0.254) (filled_areas_thickness no)
